Commit message: Added anymal and supraped

File: examples/99-robot_graphics/HRP4c.urdf (robot description, URDF)
Before this commit: robot HRP4C, 37 links, 36 joints
Links:
- link LL_KOSY_L1: mass 2.7752200000 -> 1
- link LL_KOSY_L23: mass 2.2450500000 -> 1
- link LL_KOSY_L4: mass 2.6274500000 -> 1; geometry visual mesh filename=../../../../examples/99-robot_graphics/HRP4c/graphics/L_HIP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
- link LL_KOSY_L56: mass 5.7035400000 -> 1; geometry visual mesh filename=../../../../examples/99-robot_graphics/HRP4c/graphics/L_KNE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
- link LL_ankle: mass 0.3906700000 -> 1
- link LL_foot: mass 1.4241951000 -> 1; geometry visual mesh filename=../../../../examples/99-robot_graphics/HRP4c/graphics/L_ANK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
- link RL_KOSY_L23: mass 2.2450500000 -> 1
- link RL_KOSY_L4: mass 2.6274500000 -> 1; geometry visual mesh filename=../../../../examples/99-robot_graphics/HRP4c/graphics/R_HIP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
- link RL_KOSY_L56: mass 5.7035400000 -> 1; geometry visual mesh filename=../../../../examples/99-robot_graphics/HRP4c/graphics/R_KNE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
- link RL_ankle: mass 0.3906700000 -> 1
- link RL_foot: mass 1.4241951000 -> 1; geometry visual mesh filename=../../../../examples/99-robot_graphics/HRP4c/graphics/R_ANK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
- link hip_base: mass 5.6174600000 -> 1; geometry visual mesh filename=../../../../examples/99-robot_graphics/HRP4c/graphics/WAIST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
- link la_end_effector: mass 0.1 -> 1; geometry visual mesh filename=../../../../examples/99-robot_graphics/HRP4c/graphics/L_WRI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
- link la_link1: mass 2.2396100000 -> 1; geometry visual mesh filename=../../../../examples/99-robot_graphics/HRP4c/graphics/L_SHO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
- link la_link2: geometry visual mesh filename=../../../../examples/99-robot_graphics/HRP4c/graphics/L_SHO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
- link la_link3: mass 2.3629100000 -> 1; geometry visual mesh filename=../../../../examples/99-robot_graphics/HRP4c/graphics/L_SHO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
- link la_link4: mass 0.7187000000 -> 1; geometry visual mesh filename=../../../../examples/99-robot_graphics/HRP4c/graphics/L_ELB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
- link la_link5: mass 2.2786200000 -> 1; geometry visual mesh filename=../../../../examples/99-robot_graphics/HRP4c/graphics/L_WRI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
- link la_link6: mass 0.2863747200 -> 1
- link neck_link1: mass 0.3364400000 -> 1
- link neck_link2: mass 2.4522900000 -> 1; geometry visual mesh filename=../../../../examples/99-robot_graphics/HRP4c/graphics/Helme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; visual mesh filename=../../../../examples/99-robot_graphics/HRP4c/graphics/NECK_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
- link ra_end_effector: mass 0.1 -> 1; geometry visual mesh filename=../../../../examples/99-robot_graphics/HRP4c/graphics/R_WRI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
- link ra_link1: mass 2.2396100000 -> 1; geometry visual mesh filename=../../../../examples/99-robot_graphics/HRP4c/graphics/R_SHO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
- link ra_link2: mass 1.0993800000 -> 1; geometry visual mesh filename=../../../../examples/99-robot_graphics/HRP4c/graphics/R_SHO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
- link ra_link3: mass 2.3629100000 -> 1; geometry visual mesh filename=../../../../examples/99-robot_graphics/HRP4c/graphics/R_SHO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
- link ra_link4: mass 0.7187000000 -> 1; geometry visual mesh filename=../../../../examples/99-robot_graphics/HRP4c/graphics/R_ELB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
- link ra_link5: mass 2.2786200000 -> 1; geometry visual mesh filename=../../../../examples/99-robot_graphics/HRP4c/graphics/R_WRI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
- link ra_link6: mass 0.2863747200 -> 1
- link trunk: mass 18.9794300000 -> 1; geometry visual mesh filename=../../../../examples/99-robot_graphics/HRP4c/graphics/CHEST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
- link trunk_rz: mass 18.9794300000 -> 1; geometry visual mesh filename=../../../../examples/99-robot_graphics/HRP4c/graphics/CHEST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
Joints:
- joint j1: limit lower=-1.5708 upper=0.7854 effort=176 velocity=1.9199 -> lower=-3.1415 upper=3.1415 effort=176 velocity=1.9199
- joint j10: limit lower=-1.8326 upper=1.8326 effort=165 velocity=3.0718 -> lower=0.5 upper=3.1415 effort=165 velocity=3.0718
- joint j11: limit lower=-0.3403 upper=0.3403 effort=50 velocity=2.0944 -> lower=-3.1415 upper=3.1415 effort=50 velocity=2.0944
- joint j12: limit lower=-0.7854 upper=0.7854 effort=165 velocity=3.0718 -> lower=-3.1415 upper=3.1415 effort=165 velocity=3.0718; origin xyz=-0.0000000000 0.0000000000 -0.0200000 rpy=0 0 0 -> xyz=0 0 0 rpy=0 0 0
- joint j13: limit lower=-2.0944 upper=2.0944 effort=100 velocity=2.7402 -> lower=-3.1415 upper=3.1415 effort=100 velocity=2.7402
- joint j14: limit lower=-2.0944 upper=2.0944 effort=100 velocity=2.7402 -> lower=-3.1415 upper=3.1415 effort=100 velocity=2.7402
- joint j15: limit lower=-2.0944 upper=2.0944 effort=100 velocity=2.7402 -> lower=-1.5717 upper=1.5717 effort=100 velocity=2.7402
- joint j16: limit lower=-0.2618 upper=3.1416 effort=100 velocity=2.7402 -> lower=-1.5717 upper=-0.2 effort=100 velocity=2.7402; origin xyz=0.0539500000 0.0000000000 0.0000000000 rpy=0.0000000000 0.0000000000 0 -> xyz=0 0.0000000000 0.0000000000 rpy=0.0000000000 0.0000000000 0
- joint j17: limit lower=-1.8326 upper=1.8326 effort=40 velocity=2.0944 -> lower=-1.5717 upper=1.5717 effort=40 velocity=2.0944
- joint j18: limit lower=0 upper=2.5831 effort=40 velocity=2.0944 -> lower=-3.1415 upper=-0.05 effort=40 velocity=2.0944
- joint j19: limit lower=-2.5307 upper=2.0595 effort=40 velocity=2.0944 -> lower=-1.5717 upper=1.5717 effort=40 velocity=2.0944; origin xyz=0.0000 -0.035  -0.21 rpy=-0.0871 0 0 -> xyz=0.0000 -0.035  -0.21 rpy=-0.177 0 0
- joint j2: limit lower=-2.0071 upper=1.5708 effort=100 velocity=2.7402 -> lower=-3.1415 upper=3.1415 effort=100 velocity=2.7402; origin xyz=-0.0000000000 -0.0350000000 -0.1200000000 rpy=0 0 0 -> xyz=0 0 0 rpy=0 0 0
- joint j20: limit lower=-1.8326 upper=1.8326 effort=35 velocity=2.0944 -> lower=-1.5717 upper=1.5717 effort=40 velocity=2.0944
- joint j21: limit lower=-2.0944 upper=2.0944 effort=100 velocity=2.7402 -> lower=-1.5717 upper=1.5717 effort=100 velocity=2.7402
- joint j22: limit lower=-0.2618 upper=3.1416 effort=100 velocity=2.7402 -> lower=0.2 upper=1.5717 effort=100 velocity=2.7402
- joint j23: limit lower=-1.8326 upper=1.8326 effort=40 velocity=2.0944 -> lower=-1.5717 upper=1.5717 effort=40 velocity=2.0944
- joint j24: axis 0 0 1 -> 0 1 0; limit lower=0 upper=2.5831 effort=40 velocity=2.0944 -> lower=-1.5717 upper=-0.05 effort=40 velocity=2.0944
- joint j25: limit lower=-2.5307 upper=2.0595 effort=40 velocity=2.0944 -> lower=-1.5717 upper=1.5717 effort=40 velocity=2.0944
- joint j26: limit lower=-1.8326 upper=1.8326 effort=40 velocity=2.0944 -> lower=-1.5717 upper=1.5717 effort=40 velocity=2.0944
- joint j27: limit lower=-1.5708 upper=1.5708 effort=8.4 velocity=4.7124 -> lower=-3.1415 upper=3.1415 effort=8.4 velocity=4.7124
- joint j28: limit lower=-0.5236 upper=1.5708 effort=8.4 velocity=4.7124 -> lower=-3.1415 upper=3.1415 effort=8.4 velocity=4.7124; origin xyz=-0.035 0 0.05 -> xyz=0 0 0
- joint j3: limit lower=-2.0944 upper=2.0944 effort=100 velocity=2.7402 -> lower=-3.1415 upper=3.1415 effort=100 velocity=2.7402
- joint j4: limit lower=-1.8326 upper=1.8326 effort=165 velocity=3.0718 -> lower=0.5 upper=3.1415 effort=165 velocity=3.0718
- joint j5: limit lower=-0.3403 upper=0.3403 effort=50 velocity=2.0944 -> lower=-3.1415 upper=3.1415 effort=50 velocity=2.0944
- joint j6: limit lower=-0.7804 upper=0.7804 effort=165 velocity=3.0718 -> lower=-3.1415 upper=3.1415 effort=165 velocity=3.0718
- joint j7: limit lower=-0.7804 upper=1.5708 effort=176 velocity=1.9199 -> lower=-3.1415 upper=3.1415 effort=176 velocity=1.9199
- joint j8: limit lower=-2.0071 upper=1.5708 effort=100 velocity=2.7402 -> lower=-3.1415 upper=3.1415 effort=100 velocity=2.7402
- joint j9: limit lower=-2.0944 upper=2.0944 effort=100 velocity=2.7402 -> lower=-3.1415 upper=3.1415 effort=100 velocity=2.7402
- joint j_lhand_revolute: limit lower=-1.8326 upper=1.8326 effort=35 velocity=2.0944 -> lower=-1.5717 upper=1.5717 effort=35 velocity=2.0944
- joint j_rhand_revolute: axis 0 0 1 -> 1 0 0; limit lower=-1.8326 upper=1.8326 effort=35 velocity=2.0944 -> lower=-1.5717 upper=1.5717 effort=40 velocity=2.0944
